File: controller/codec.sch (KiCad schematic (older format))
At the start: 157 parts, among them J14 Left, J15 Right, J16 Conn_01x03_Male, J17 Conn_01x03_Male, J18 ch5, J19 ch6, J20 ch1, J21 ch2, J22 ch3, J23 ch4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

Commit message: update components
Parts:
- added C141, C142: 0.1, Capacitor_SMD:C_0603_1608Metric_Pad1.08x0.95mm_HandSolder, symbol Device:C
- C11, C15: footprint Capacitor_SMD:CP_Elec_5x5.8 -> Capacitor_SMD:CP_Elec_6.3x5.3
- C19, C20, C23, C30, C33, C34, C35, C36, C37, C70, C71, C72, C74, C75, C76: footprint Capacitor_SMD:C_0603_1608Metric_Pad1.08x0.95mm_HandSolder -> Capacitor_SMD:C_0805_2012Metric_Pad1.18x1.45mm_HandSolder
- C25, C32: value 10hF -> 100pF
- C26: value 10hF -> 10uF; footprint Capacitor_SMD:C_0603_1608Metric_Pad1.08x0.95mm_HandSolder -> Capacitor_SMD:C_0805_2012Metric_Pad1.18x1.45mm_HandSolder
Connections:
- net +3.3VA: now also C141.1, C142.1
- net BAL_IN_L_N: now also U7.60 (ADC2RN); no longer U7.58 (ADC2LN)
- net BAL_IN_L_P: now also U7.59 (ADC2RP); no longer U7.57 (ADC2LP)
- net BAL_IN_R_N: now also U7.58 (ADC2LN); no longer U7.60 (ADC2RN)
- net BAL_IN_R_P: now also U7.57 (ADC2LP); no longer U7.59 (ADC2RP)
- net GNDA: now also C141.2, C142.2
Other:
- moved on the sheet: C102, C63, C64, C65, C66, C67, C68, C69, C73, C77, C78, C79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
