File: controller/dsp.sch (KiCad schematic (older format))
At the start: 73 parts, among them J1 PRG, J27 TP, J28 TP, J29 TP, J30 TP, J31 TP, J32 TP, J33 TP, J34 TP, J35 TP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

Commit message: Fix misc issues
Parts:
- added C?: 0.1, Capacitor_SMD:C_0603_1608Metric_Pad1.08x0.95mm_HandSolder, symbol Device:C
- added NT?: NT1, symbol Device:Net-Tie_2
Connections:
- net +3V3: now also NT?.2
- net GND: now also C?.2
- net VPP: now also C?.1, NT?.1
Changed lines of the file:
@@
 Connection ~ 6600 9100
 Connection ~ 6600 8700
+$Comp
+L Device:Net-Tie_2 NT?
+U 1 1 614731D0
+P 12950 2800
+F 0 "NT?" V 12996 2756 50  0000 R CNN
+F 1 "NT1" V 12905 2756 50  0000 R CNN
+F 2 "" H 12950 2800 50  0001 C CNN
+F 3 "~" H 12950 2800 50  0001 C CNN
+	1    12950 2800
+	0    -1   -1   0
+$EndComp
+Wire Wire Line
+	13300 3000 12950 3000
+Connection ~ 13300 3000
+Wire Wire Line
+	13300 2600 12950 2600
+Connection ~ 13300 2600
+Wire Wire Line
+	12950 2700 12950 2600
+Wire Wire Line
+	12950 2900 12950 3000
+$Comp
+L Device:C C?
+U 1 1 61572478
+P 12950 3250
+AR Path="/60CBC38F/61572478" Ref="C?"  Part="1"
+AR Path="/60BF255D/61572478" Ref="C?"  Part="1"
+F 0 "C?" V 12900 3350 50  0000 C CNN
+F 1 "0.1" V 13000 3400 50  0000 C CNN
+F 2 "Capacitor_SMD:C_0603_1608Metric_Pad1.08x0.95mm_HandSolder" H 12988 3100 50  0001 C CNN
+F 3 "~" H 12950 3250 50  0001 C CNN
+	1    12950 3250
+	1    0    0    -1
+$EndComp
+Wire Wire Line
+	12950 3000 12950 3100
+Connection ~ 12950 3000
+Wire Wire Line
+	12950 3500 13450 3500
+Wire Wire Line
+	12950 3400 12950 3500
 $EndSCHEMATC
