File: controller/ps.sch (KiCad schematic (older format))
At the start: 57 parts, among them J10 PRI_TRF_L, J11 PRI_TRF_N, J12 SEC_OUT_L, J13 SEC_OUT_N, J6 MAIN_PWR_L, J7 MAIN_PWR_N, J8 SEC_TRF_L, J9 SEC_TRF_N, Q2 BC846A, U1 LM2596S-ADJ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

Commit message: update components
Parts:
- removed U19, U20: TCM809, Package_TO_SOT_SMD:SOT-23, symbol Power_Supervisor:TCM809
- added L2: FB, Inductor_SMD:L_0805_2012Metric_Pad1.15x1.40mm_HandSolder, symbol pspice:INDUCTOR
- added U19, U20: MCP130-xxxxTT, Package_TO_SOT_SMD:SOT-23, symbol Power_Supervisor:MCP130-xxxxTT
- R158: value R -> 1K3
- R159: value R -> 11K
- R160: value R -> 360R
- R161: value R -> 1K1
- R162: value R -> 620R
- R163: value R -> 1K
Connections:
- net +3V3: now also U19.2 (VDD)
- net +5V: now also U20.2 (VDD)
- net GND: now also L2.1, U19.3 (VSS), U20.3 (VSS)
- net GNDA: now also L2.2
- net WR_BACK: now also U20.1 (~RST)
- net nRST: now also U19.1 (~RST)
Changed lines of the file:
@@
 	1    0    0    -1
 $EndComp
-Text HLabel 10300 1900 2    50   Input ~ 0
+Text HLabel 10200 1900 2    50   Input ~ 0
 WR_BACK
-Text HLabel 9050 1900 2    50   Input ~ 0
+Text HLabel 8950 1900 2    50   Input ~ 0
 nRST
-$Comp
-L Power_Supervisor:TCM809 U19
-U 1 1 631691FD
-P 8650 1900
-F 0 "U19" H 8420 1946 50  0000 R CNN
-F 1 "TCM809" H 8420 1855 50  0000 R CNN
-F 2 "Package_TO_SOT_SMD:SOT-23" H 8250 2050 50  0001 C CNN
-F 3 "http://ww1.microchip.com/downloads/en/DeviceDoc/21661E.pdf" H 8350 2150 50  0001 C CNN
-	1    8650 1900
-	1    0    0    -1
-$EndComp
 $Comp
 L power:+3.3V #PWR0244
@@
 $EndComp
 $Comp
-L Power_Supervisor:TCM809 U20
-U 1 1 6317A7EA
-P 9900 1900
-F 0 "U20" H 9670 1946 50  0000 R CNN
-F 1 "TCM809" H 9670 1855 50  0000 R CNN
-F 2 "Package_TO_SOT_SMD:SOT-23" H 9500 2050 50  0001 C CNN
-F 3 "http://ww1.microchip.com/downloads/en/DeviceDoc/21661E.pdf" H 9600 2150 50  0001 C CNN
-	1    9900 1900
-	1    0    0    -1
-$EndComp
-$Comp
 L power:GND #PWR0246
 U 1 1 6317A7F6
@@
 	8550 1500 8550 1400
 Wire Wire Line
-	8950 1900 9050 1900
+	8850 1900 8950 1900
 Wire Wire Line
 	8550 2400 8550 2300
@@
 	9800 2400 9800 2300
 Wire Wire Line
-	10200 1900 10300 1900
+	10100 1900 10200 1900
 Wire Wire Line
 	9800 1500 9800 1400
@@
 P 5500 3400
 F 0 "R159" V 5400 3400 50  0000 C CNN
-F 1 "R" V 5500 3400 50  0000 C CNN
+F 1 "11K" V 5500 3400 50  0000 C CNN
 F 2 "Resistor_SMD:R_0603_1608Metric_Pad0.98x0.95mm_HandSolder" V 5430 3400 50  0001 C CNN
 F 3 "~" H 5500 3400 50  0001 C CNN
@@
 P 5150 3850
 F 0 "R158" V 5050 3850 50  0000 C CNN
-F 1 "R" V 5150 3850 50  0000 C CNN
+F 1 "1K3" V 5150 3850 50  0000 C CNN
 F 2 "Resistor_SMD:R_0603_1608Metric_Pad0.98x0.95mm_HandSolder" V 5080 3850 50  0001 C CNN
 F 3 "~" H 5150 3850 50  0001 C CNN
@@
 P 8650 3700
 F 0 "R160" V 8550 3700 50  0000 C CNN
-F 1 "R" V 8650 3700 50  0000 C CNN
+F 1 "360R" V 8650 3700 50  0000 C CNN
 F 2 "Resistor_SMD:R_0603_1608Metric_Pad0.98x0.95mm_HandSolder" V 8580 3700 50  0001 C CNN
 F 3 "~" H 8650 3700 50  0001 C CNN
@@
 P 8650 4100
 F 0 "R161" V 8550 4100 50  0000 C CNN
-F 1 "R" V 8650 4100 50  0000 C CNN
+F 1 "1K1" V 8650 4100 50  0000 C CNN
 F 2 "Resistor_SMD:R_0603_1608Metric_Pad0.98x0.95mm_HandSolder" V 8580 4100 50  0001 C CNN
 F 3 "~" H 8650 4100 50  0001 C CNN
@@
 P 8650 5200
 F 0 "R162" V 8550 5200 50  0000 C CNN
-F 1 "R" V 8650 5200 50  0000 C CNN
+F 1 "620R" V 8650 5200 50  0000 C CNN
 F 2 "Resistor_SMD:R_0603_1608Metric_Pad0.98x0.95mm_HandSolder" V 8580 5200 50  0001 C CNN
 F 3 "~" H 8650 5200 50  0001 C CNN
@@
 P 8650 5600
 F 0 "R163" V 8550 5600 50  0000 C CNN
-F 1 "R" V 8650 5600 50  0000 C CNN
+F 1 "1K" V 8650 5600 50  0000 C CNN
 F 2 "Resistor_SMD:R_0603_1608Metric_Pad0.98x0.95mm_HandSolder" V 8580 5600 50  0001 C CNN
 F 3 "~" H 8650 5600 50  0001 C CNN
@@
 	1    0    0    -1
 $EndComp
+$Comp
+L Power_Supervisor:MCP130-xxxxTT U19
+U 1 1 60E64E14
+P 8550 1900
+F 0 "U19" H 8450 1950 50  0000 R CNN
+F 1 "MCP130-xxxxTT" H 9200 1550 50  0000 R CNN
+F 2 "Package_TO_SOT_SMD:SOT-23" H 9150 1550 50  0001 C CNN
+F 3 "http://ww1.microchip.com/downloads/en/DeviceDoc/11184d.pdf" H 8550 1900 50  0001 C CNN
+	1    8550 1900
+	1    0    0    -1
+$EndComp
+$Comp
+L Power_Supervisor:MCP130-xxxxTT U20
+U 1 1 60E778D1
+P 9800 1900
+F 0 "U20" H 9700 1950 50  0000 R CNN
+F 1 "MCP130-xxxxTT" H 10450 1550 50  0000 R CNN
+F 2 "Package_TO_SOT_SMD:SOT-23" H 10400 1550 50  0001 C CNN
+F 3 "http://ww1.microchip.com/downloads/en/DeviceDoc/11184d.pdf" H 9800 1900 50  0001 C CNN
+	1    9800 1900
+	1    0    0    -1
+$EndComp
+$Comp
+L power:GND #PWR0195
+U 1 1 614186E1
+P 4500 6250
+F 0 "#PWR0195" H 4500 6000 50  0001 C CNN
+F 1 "GND" H 4505 6077 50  0000 C CNN
+F 2 "" H 4500 6250 50  0001 C CNN
+F 3 "" H 4500 6250 50  0001 C CNN
+	1    4500 6250
+	1    0    0    -1
+$EndComp
+$Comp
+L power:GNDA #PWR0201
+U 1 1 614186E7
+P 5200 6250
+F 0 "#PWR0201" H 5200 6000 50  0001 C CNN
+F 1 "GNDA" H 5205 6077 50  0000 C CNN
+F 2 "" H 5200 6250 50  0001 C CNN
+F 3 "" H 5200 6250 50  0001 C CNN
+	1    5200 6250
+	1    0    0    -1
+$EndComp
+$Comp
+L pspice:INDUCTOR L2
+U 1 1 6141EE6F
+P 4850 6100
+F 0 "L2" H 4850 6315 50  0000 C CNN
+F 1 "FB" H 4850 6224 50  0000 C CNN
+F 2 "Inductor_SMD:L_0805_2012Metric_Pad1.15x1.40mm_HandSolder" H 4850 6100 50  0001 C CNN
+F 3 "~" H 4850 6100 50  0001 C CNN
+	1    4850 6100
+	1    0    0    -1
+$EndComp
+Wire Wire Line
+	5200 6250 5200 6100
+Wire Wire Line
+	5200 6100 5100 6100
+Wire Wire Line
+	4600 6100 4500 6100
+Wire Wire Line
+	4500 6100 4500 6250
 $EndSCHEMATC

Commit message: Fix misc issues
Parts:
- removed C10: 100uF, Capacitor_SMD:CP_Elec_6.3x7.7, symbol Device:CP
- removed C9: 0.1, Capacitor_SMD:C_0805_2012Metric_Pad1.18x1.45mm_HandSolder, symbol Device:C
- removed D4: 1N4148, Diode_SMD:D_SOD-323_HandSoldering, symbol Device:D
- removed D5: 12V, Diode_SMD:D_SOD-123F, symbol Device:D_Zener
- removed Q2: BC846A, Package_TO_SOT_SMD:SOT-23, symbol Device:Q_NPN_BEC
- removed R27: 1K, Resistor_SMD:R_0603_1608Metric_Pad0.98x0.95mm_HandSolder, symbol Device:R
- removed R28: 100, Resistor_SMD:R_0603_1608Metric_Pad0.98x0.95mm_HandSolder, symbol Device:R
- removed U6: SFH6186-4T, Package_SO:SO-4_7.6x3.6mm_P2.54mm, symbol Isolator:SFH617A-1X001
- added R?: 330/1W, Resistor_THT:R_Axial_DIN0414_L11.9mm_D4.5mm_P15.24mm_Horizontal, symbol Device:R
- added U6: MOC3083M, symbol Relay_SolidState:MOC3083M
- C6: value 0.1uF/400V -> 0.01uF/630V
- R158: value 1K3 -> 2K
- R26: value 2K2/1W -> 56/2W
Connections:
- net +3V3: now also U6.1
- net MAIN_TRF_CTRL: now also U6.2
- net at C6.2, D3.1 (A1), J10.1 (Pin_1): now also R?.2
- net at D3.3 (G): now also R?.1, U6.4
- net at R26.1: now also U6.6
Changed lines of the file:
@@
 P 2400 2100
 F 0 "C6" H 2515 2146 50  0000 L CNN
-F 1 "0.1uF/400V" H 2515 2055 50  0000 L CNN
+F 1 "0.01uF/630V" H 2515 2055 50  0000 L CNN
 F 2 "Capacitor_THT:C_Disc_D8.0mm_W5.0mm_P10.00mm" H 2438 1950 50  0001 C CNN
 F 3 "~" H 2400 2100 50  0001 C CNN
@@
 P 3350 1500
 F 0 "R26" V 3143 1500 50  0000 C CNN
-F 1 "2K2/1W" V 3234 1500 50  0000 C CNN
+F 1 "56/2W" V 3234 1500 50  0000 C CNN
 F 2 "Resistor_THT:R_Axial_DIN0414_L11.9mm_D4.5mm_P15.24mm_Horizontal" V 3280 1500 50  0001 C CNN
 F 3 "~" H 3350 1500 50  0001 C CNN
@@
 Wire Wire Line
 	2850 1500 3200 1500
-$Comp
-L Device:D D4
-U 1 1 60C0A6FE
-P 3800 1500
-F 0 "D4" H 3800 1283 50  0000 C CNN
-F 1 "1N4148" H 3800 1374 50  0000 C CNN
-F 2 "Diode_SMD:D_SOD-323_HandSoldering" H 3800 1500 50  0001 C CNN
-F 3 "~" H 3800 1500 50  0001 C CNN
-	1    3800 1500
-	-1   0    0    1
-$EndComp
-Wire Wire Line
-	3500 1500 3650 1500
-$Comp
-L Device:C C9
-U 1 1 60C0B755
-P 4100 1950
-F 0 "C9" H 4215 1996 50  0000 L CNN
-F 1 "0.1" H 4215 1905 50  0000 L CNN
-F 2 "Capacitor_SMD:C_0805_2012Metric_Pad1.18x1.45mm_HandSolder" H 4138 1800 50  0001 C CNN
-F 3 "~" H 4100 1950 50  0001 C CNN
-	1    4100 1950
-	1    0    0    -1
-$EndComp
-$Comp
-L Device:CP C10
-U 1 1 60C0BEBC
-P 4450 1950
-F 0 "C10" H 4568 1996 50  0000 L CNN
-F 1 "100uF" H 4568 1905 50  0000 L CNN
-F 2 "Capacitor_SMD:CP_Elec_6.3x7.7" H 4488 1800 50  0001 C CNN
-F 3 "~" H 4450 1950 50  0001 C CNN
-	1    4450 1950
-	1    0    0    -1
-$EndComp
-$Comp
-L Device:D_Zener D5
-U 1 1 60C0C76A
-P 4850 1950
-F 0 "D5" V 4804 2030 50  0000 L CNN
-F 1 "12V" V 4895 2030 50  0000 L CNN
-F 2 "Diode_SMD:D_SOD-123F" H 4850 1950 50  0001 C CNN
-F 3 "~" H 4850 1950 50  0001 C CNN
-	1    4850 1950
-	0    1    1    0
-$EndComp
-Wire Wire Line
-	3950 1500 4100 1500
-Wire Wire Line
-	4850 1500 4850 1800
-Wire Wire Line
-	4100 1800 4100 1500
-Connection ~ 4100 1500
-Wire Wire Line
-	4100 1500 4450 1500
-Connection ~ 4450 1500
-Wire Wire Line
-	4450 1500 4850 1500
-Wire Wire Line
-	4850 2300 4850 2100
-Wire Wire Line
-	4450 1500 4450 1800
-Wire Wire Line
-	4100 2100 4100 2300
-Wire Wire Line
-	2850 2300 3350 2300
-Connection ~ 4100 2300
-Wire Wire Line
-	4100 2300 4450 2300
-Wire Wire Line
-	4450 2100 4450 2300
-Connection ~ 4450 2300
-Wire Wire Line
-	4450 2300 4850 2300
-$Comp
-L Device:R R28
-U 1 1 60C103E8
-P 3600 1650
-F 0 "R28" V 3500 1650 50  0000 C CNN
-F 1 "100" V 3600 1650 50  0000 C CNN
-F 2 "Resistor_SMD:R_0603_1608Metric_Pad0.98x0.95mm_HandSolder" V 3530 1650 50  0001 C CNN
-F 3 "~" H 3600 1650 50  0001 C CNN
-	1    3600 1650
-	0    1    1    0
-$EndComp
-$Comp
-L Device:R R27
-U 1 1 60C122DF
-P 3350 1950
-F 0 "R27" V 3250 1950 50  0000 C CNN
-F 1 "1K" V 3350 1950 50  0000 C CNN
-F 2 "Resistor_SMD:R_0603_1608Metric_Pad0.98x0.95mm_HandSolder" V 3280 1950 50  0001 C CNN
-F 3 "~" H 3350 1950 50  0001 C CNN
-	1    3350 1950
-	1    0    0    -1
-$EndComp
-Wire Wire Line
-	3350 1650 3350 1800
-Wire Wire Line
-	3350 2100 3350 2300
-$Comp
-L Device:Q_NPN_BEC Q2
-U 1 1 60C167F3
-P 5450 1450
-F 0 "Q2" H 5641 1404 50  0000 L CNN
-F 1 "BC846A" H 5641 1495 50  0000 L CNN
-F 2 "Package_TO_SOT_SMD:SOT-23" H 5650 1550 50  0001 C CNN
-F 3 "~" H 5450 1450 50  0001 C CNN
-	1    5450 1450
-	-1   0    0    -1
-$EndComp
-Connection ~ 3350 2300
-Wire Wire Line
-	3350 2300 4100 2300
-Wire Wire Line
-	3750 1650 5350 1650
-Wire Wire Line
-	3350 1650 3450 1650
-Wire Wire Line
-	5350 1250 4450 1250
-Wire Wire Line
-	4450 1250 4450 1500
-$Comp
-L Isolator:SFH617A-1X001 U6
-U 1 1 60C221BE
-P 6150 1350
-F 0 "U6" H 6150 1675 50  0000 C CNN
-F 1 "SFH6186-4T" H 6150 1584 50  0000 C CNN
-F 2 "Package_SO:SO-4_7.6x3.6mm_P2.54mm" H 5950 1150 50  0001 L CIN
-F 3 "http://www.vishay.com/docs/83740/sfh617a.pdf" H 6150 1350 50  0001 L CNN
-	1    6150 1350
-	-1   0    0    -1
-$EndComp
-Wire Wire Line
-	5850 1250 5350 1250
-Connection ~ 5350 1250
-Wire Wire Line
-	5850 1450 5650 1450
-Wire Wire Line
-	6450 1450 6850 1450
+Wire Wire Line
+	4400 1700 4800 1700
 $Comp
 L Connector:Conn_01x01_Male J12
@@
 	1    0    0    -1
 $EndComp
-Text HLabel 6850 1450 2    50   Input ~ 0
+Text HLabel 4800 1700 2    50   Input ~ 0
 MAIN_TRF_CTRL
 $Comp
@@
 Wire Wire Line
 	1600 4600 2000 4600
-Wire Wire Line
-	3000 1850 3150 1850
-Wire Wire Line
-	3150 1850 3150 1650
-Wire Wire Line
-	3150 1650 3350 1650
-Connection ~ 3350 1650
 $Comp
 L power:+3.3VA #PWR0187
@@
 L power:+3.3V #PWR0266
 U 1 1 635ACB53
-P 6650 1200
-F 0 "#PWR0266" H 6650 1050 50  0001 C CNN
-F 1 "+3.3V" H 6665 1373 50  0000 C CNN
-F 2 "" H 6650 1200 50  0001 C CNN
-F 3 "" H 6650 1200 50  0001 C CNN
-	1    6650 1200
-	1    0    0    -1
-$EndComp
-Wire Wire Line
-	6650 1250 6650 1200
-Wire Wire Line
-	6450 1250 6650 1250
+P 4600 1450
+F 0 "#PWR0266" H 4600 1300 50  0001 C CNN
+F 1 "+3.3V" H 4615 1623 50  0000 C CNN
+F 2 "" H 4600 1450 50  0001 C CNN
+F 3 "" H 4600 1450 50  0001 C CNN
+	1    4600 1450
+	1    0    0    -1
+$EndComp
+Wire Wire Line
+	4600 1500 4600 1450
+Wire Wire Line
+	4400 1500 4600 1500
 $Comp
 L power:GND #PWR0135
@@
 P 5150 3850
 F 0 "R158" V 5050 3850 50  0000 C CNN
-F 1 "1K3" V 5150 3850 50  0000 C CNN
+F 1 "2K" V 5150 3850 50  0000 C CNN
 F 2 "Resistor_SMD:R_0603_1608Metric_Pad0.98x0.95mm_HandSolder" V 5080 3850 50  0001 C CNN
 F 3 "~" H 5150 3850 50  0001 C CNN
@@
 Wire Wire Line
 	4500 6100 4500 6250
+$Comp
+L Relay_SolidState:MOC3083M U6
+U 1 1 614D1E72
+P 4100 1600
+F 0 "U6" H 4100 1925 50  0000 C CNN
+F 1 "MOC3083M" H 4100 1834 50  0000 C CNN
+F 2 "" H 3900 1400 50  0001 L CIN
+F 3 "https://www.onsemi.com/pub/Collateral/MOC3083M-D.PDF" H 4100 1600 50  0001 L CNN
+	1    4100 1600
+	-1   0    0    -1
+$EndComp
+$Comp
+L Device:R R?
+U 1 1 61538D39
+P 3300 2100
+F 0 "R?" V 3093 2100 50  0000 C CNN
+F 1 "330/1W" V 3184 2100 50  0000 C CNN
+F 2 "Resistor_THT:R_Axial_DIN0414_L11.9mm_D4.5mm_P15.24mm_Horizontal" V 3230 2100 50  0001 C CNN
+F 3 "~" H 3300 2100 50  0001 C CNN
+	1    3300 2100
+	1    0    0    -1
+$EndComp
+Wire Wire Line
+	3000 1850 3300 1850
+Wire Wire Line
+	3500 1500 3800 1500
+Wire Wire Line
+	2850 2300 3300 2300
+Wire Wire Line
+	3300 2300 3300 2250
+Wire Wire Line
+	3300 1950 3300 1850
+Connection ~ 3300 1850
+Wire Wire Line
+	3300 1850 3300 1700
+Wire Wire Line
+	3300 1700 3800 1700
 $EndSCHEMATC
