File: amp_board/amplifier.sch (KiCad schematic (older format))
At the start: 81 parts, among them J1 AUDIO_IN, J2 +VDC, J3 COM, J4 -VDC, J5 OUT_CTL, J6 SPK_POS, J7 SPK_NEG, Q1 BC846, Q10 BC850, Q11 2SK135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

Commit message: update xformer soft startup
Parts:
- added C19, C20: 22pF, Resistor_SMD:R_0805_2012Metric_Pad1.20x1.40mm_HandSolder, symbol pspice:CAP
- added C21, C22: 330nF, Capacitor_SMD:C_1206_3216Metric_Pad1.33x1.80mm_HandSolder, symbol pspice:CAP
Connections:
- net +VDC: now also C19.1, C21.1
- net -VDC: now also C20.2, C22.2
- net at C11.2, C9.1, D2.1 (K)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: now also C22.1
- net at Q5.3 (C), R12.2: now also C19.2
- net at Q6.3 (C), R13.1: now also C20.1
- net at C10.1, C8.2, D1.2 (A)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: now also C21.2
Other:
- moved on the sheet: R12
Changed lines of the file:
@@
 U 1 1 60B42D1B
 P 4150 4900
-F 0 "R1" H 4200 4950 50  0000 L CNN
+F 0 "R1" V 4050 4850 50  0000 L CNN
 F 1 "27K" V 4150 4850 50  0000 L CNN
 F 2 "Resistor_SMD:R_0603_1608Metric_Pad0.98x0.95mm_HandSolder" V 4080 4900 50  0001 C CNN
@@
 U 1 1 60B7CAE8
 P 4450 5450
-F 0 "R3" H 4520 5496 50  0000 L CNN
+F 0 "R3" V 4350 5400 50  0000 L CNN
 F 1 "10R" V 4450 5400 50  0000 L CNN
 F 2 "Resistor_SMD:R_0603_1608Metric_Pad0.98x0.95mm_HandSolder" V 4380 5450 50  0001 C CNN
@@
 U 1 1 60BD91B5
 P 10400 4500
-F 0 "R27" H 10450 4550 50  0000 L CNN
+F 0 "R27" V 10300 4450 50  0000 L CNN
 F 1 "R22" V 10400 4450 50  0000 L CNN
 F 2 "Resistor_THT:R_Axial_Power_L38.0mm_W9.0mm_P40.64mm" V 10330 4500 50  0001 C CNN
@@
 U 1 1 60BDA168
 P 11100 4500
-F 0 "R29" H 11150 4550 50  0000 L CNN
+F 0 "R29" V 11000 4450 50  0000 L CNN
 F 1 "R22" V 11100 4450 50  0000 L CNN
 F 2 "Resistor_THT:R_Axial_Power_L38.0mm_W9.0mm_P40.64mm" V 11030 4500 50  0001 C CNN
@@
 U 1 1 60BDDD66
 P 10400 4900
-F 0 "R28" H 10450 4950 50  0000 L CNN
+F 0 "R28" V 10300 4800 50  0000 L CNN
 F 1 "R22" V 10400 4850 50  0000 L CNN
 F 2 "Resistor_THT:R_Axial_Power_L38.0mm_W9.0mm_P40.64mm" V 10330 4900 50  0001 C CNN
@@
 U 1 1 60BDDD6C
 P 11100 4900
-F 0 "R30" H 11150 4950 50  0000 L CNN
+F 0 "R30" V 11000 4850 50  0000 L CNN
 F 1 "R22" V 11100 4850 50  0000 L CNN
 F 2 "Resistor_THT:R_Axial_Power_L38.0mm_W9.0mm_P40.64mm" V 11030 4900 50  0001 C CNN
@@
 U 1 1 60C89FD6
 P 9100 4200
-F 0 "RV1" H 9300 4100 50  0000 R CNN
+F 0 "RV1" V 9000 4250 50  0000 R CNN
 F 1 "220R" V 9100 4300 50  0000 R CNN
 F 2 "Potentiometer_THT:Potentiometer_Bourns_3296Y_Vertical" H 9100 4200 50  0001 C CNN
@@
 U 1 1 60CF8778
 P 9100 6750
-F 0 "R22" H 9170 6796 50  0000 L CNN
+F 0 "R22" V 9000 6650 50  0000 L CNN
 F 1 "82R" V 9100 6700 50  0000 L CNN
 F 2 "Resistor_SMD:R_2512_6332Metric_Pad1.40x3.35mm_HandSolder" V 9030 6750 50  0001 C CNN
@@
 U 1 1 60D5C645
 P 9100 2700
-F 0 "R21" H 9170 2746 50  0000 L CNN
+F 0 "R21" V 9000 2600 50  0000 L CNN
 F 1 "82R" V 9100 2650 50  0000 L CNN
 F 2 "Resistor_SMD:R_2512_6332Metric_Pad1.40x3.35mm_HandSolder" V 9030 2700 50  0001 C CNN
@@
 U 1 1 60D80CE5
 P 8350 3950
-F 0 "R19" H 8400 4000 50  0000 L CNN
+F 0 "R19" V 8250 3900 50  0000 L CNN
 F 1 "10K" V 8350 3900 50  0000 L CNN
 F 2 "Resistor_SMD:R_2512_6332Metric_Pad1.40x3.35mm_HandSolder" V 8280 3950 50  0001 C CNN
@@
 $EndComp
 $Comp
-L pspice:CAP C10
-U 1 1 60D85DD3
-P 8650 3950
-F 0 "C10" H 8750 4100 50  0000 L CNN
-F 1 "330nF" H 8750 3800 50  0000 L CNN
-F 2 "Capacitor_SMD:C_1206_3216Metric_Pad1.33x1.80mm_HandSolder" H 8650 3950 50  0001 C CNN
-F 3 "~" H 8650 3950 50  0001 C CNN
-	1    8650 3950
-	1    0    0    -1
-$EndComp
-$Comp
 L Device:R R20
 U 1 1 60D9FB55
 P 8350 5500
-F 0 "R20" H 8400 5550 50  0000 L CNN
+F 0 "R20" V 8250 5400 50  0000 L CNN
 F 1 "10K" V 8350 5450 50  0000 L CNN
 F 2 "Resistor_SMD:R_2512_6332Metric_Pad1.40x3.35mm_HandSolder" V 8280 5500 50  0001 C CNN
@@
 $EndComp
 Wire Wire Line
-	8800 3650 8650 3650
-Wire Wire Line
 	8350 3650 8350 3800
 Wire Wire Line
@@
 Wire Wire Line
 	8650 4250 8800 4250
-$Comp
-L Device:D_Zener D2
-U 1 1 60DF1524
-P 8650 6750
-F 0 "D2" V 8604 6830 50  0000 L CNN
-F 1 "3V9" V 8695 6830 50  0000 L CNN
-F 2 "Diode_SMD:D_SOD-123" H 8650 6750 50  0001 C CNN
-F 3 "~" H 8650 6750 50  0001 C CNN
-	1    8650 6750
-	0    1    1    0
-$EndComp
 Wire Wire Line
 	9100 6950 8650 6950
@@
 	9100 7000 9100 6950
 Connection ~ 9100 6950
-Wire Wire Line
-	8650 5800 8650 6550
 $Comp
 L Device:CP C9
@@
 $EndComp
 Wire Wire Line
-	8450 6600 8450 6550
-Wire Wire Line
-	8450 6550 8650 6550
-Connection ~ 8650 6550
-Wire Wire Line
-	8650 6550 8650 6600
-Wire Wire Line
 	8650 6950 8450 6950
 Wire Wire Line
@@
 $EndComp
 Wire Wire Line
-	8450 2850 8450 2900
-Wire Wire Line
-	8450 2900 8650 2900
-Wire Wire Line
-	8650 2900 8650 2850
-Wire Wire Line
 	9100 2500 8650 2500
 Wire Wire Line
@@
 Wire Wire Line
 	8650 2500 8450 2500
-Wire Wire Line
-	8650 2900 8650 3650
-Connection ~ 8650 2900
 Wire Wire Line
 	9100 2450 9100 2500
@@
 U 1 1 60EB94D6
 P 5650 2700
-F 0 "R4" H 5700 2750 50  0000 L CNN
+F 0 "R4" V 5550 2650 50  0000 L CNN
 F 1 "6K8" V 5650 2650 50  0000 L CNN
 F 2 "Resistor_SMD:R_0603_1608Metric_Pad0.98x0.95mm_HandSolder" V 5580 2700 50  0001 C CNN
@@
 U 1 1 60ED4471
 P 6300 2300
-F 0 "R9" H 6350 2350 50  0000 L CNN
+F 0 "R9" V 6200 2250 50  0000 L CNN
 F 1 "5K6" V 6300 2250 50  0000 L CNN
 F 2 "Resistor_SMD:R_0603_1608Metric_Pad0.98x0.95mm_HandSolder" V 6230 2300 50  0001 C CNN
@@
 L Device:R R12
 U 1 1 60F13259
-P 6800 2850
-F 0 "R12" H 6850 2900 50  0000 L CNN
-F 1 "6K8" V 6800 2800 50  0000 L CNN
-F 2 "Resistor_SMD:R_0603_1608Metric_Pad0.98x0.95mm_HandSolder" V 6730 2850 50  0001 C CNN
-F 3 "~" H 6800 2850 50  0001 C CNN
-	1    6800 2850
+P 6800 2650
+F 0 "R12" V 6700 2600 50  0000 L CNN
+F 1 "6K8" V 6800 2600 50  0000 L CNN
+F 2 "Resistor_SMD:R_0603_1608Metric_Pad0.98x0.95mm_HandSolder" V 6730 2650 50  0001 C CNN
+F 3 "~" H 6800 2650 50  0001 C CNN
+	1    6800 2650
 	1    0    0    -1
 $EndComp
@@
 Wire Wire Line
 	6650 2700 6600 2700
-Wire Wire Line
-	6800 2100 6800 2700
-Wire Wire Line
-	6650 2100 6800 2100
 Connection ~ 6650 2100
 $Comp
@@
 	6300 2050 6300 2100
 Wire Wire Line
-	6800 3000 6800 3750
-Wire Wire Line
 	6700 4150 6800 4150
 Wire Wire Line
@@
 U 1 1 60FFBCB6
 P 6800 6600
-F 0 "R13" H 6850 6650 50  0000 L CNN
+F 0 "R13" V 6700 6550 50  0000 L CNN
 F 1 "6K8" V 6800 6550 50  0000 L CNN
 F 2 "Resistor_SMD:R_0603_1608Metric_Pad0.98x0.95mm_HandSolder" V 6730 6600 50  0001 C CNN
@@
 U 1 1 60FFBCBD
 P 5650 6650
-F 0 "R5" H 5700 6700 50  0000 L CNN
+F 0 "R5" V 5550 6600 50  0000 L CNN
 F 1 "6K8" V 5650 6600 50  0000 L CNN
 F 2 "Resistor_SMD:R_0603_1608Metric_Pad0.98x0.95mm_HandSolder" V 5580 6650 50  0001 C CNN
@@
 U 1 1 60FFBCCB
 P 6250 7050
-F 0 "R8" H 6300 7100 50  0000 L CNN
+F 0 "R8" V 6150 7000 50  0000 L CNN
 F 1 "5K6" V 6250 7000 50  0000 L CNN
 F 2 "Resistor_SMD:R_0603_1608Metric_Pad0.98x0.95mm_HandSolder" V 6180 7050 50  0001 C CNN
@@
 Connection ~ 5650 6300
 Wire Wire Line
-	6800 5450 6800 6450
+	6800 5450 6800 6400
 Wire Wire Line
 	6800 6750 6800 7250
@@
 U 1 1 61179A2C
 P 8800 9500
-F 0 "C12" H 8600 9500 50  0000 C CNN
+F 0 "C12" H 8600 9600 50  0000 C CNN
 F 1 "100uF/80V" H 8650 9400 50  0000 C CNN
 F 2 "Capacitor_SMD:CP_Elec_16x17.5" H 8838 9350 50  0001 C CNN
@@
 U 1 1 61179A32
 P 8800 10000
-F 0 "C13" H 8600 10000 50  0000 C CNN
+F 0 "C13" H 8600 10100 50  0000 C CNN
 F 1 "100uF/80V" H 8650 9900 50  0000 C CNN
 F 2 "Capacitor_SMD:CP_Elec_16x17.5" H 8838 9850 50  0001 C CNN
@@
 Wire Wire Line
 	12000 5100 12300 5100
+Wire Wire Line
+	8800 3650 8650 3650
+$Comp
+L pspice:CAP C10
+U 1 1 60D85DD3
+P 8650 3950
+F 0 "C10" H 8750 4100 50  0000 L CNN
+F 1 "330nF" H 8750 3800 50  0000 L CNN
+F 2 "Capacitor_SMD:C_1206_3216Metric_Pad1.33x1.80mm_HandSolder" H 8650 3950 50  0001 C CNN
+F 3 "~" H 8650 3950 50  0001 C CNN
+	1    8650 3950
+	1    0    0    -1
+$EndComp
+$Comp
+L pspice:CAP C22
+U 1 1 61783BCB
+P 7950 6700
+F 0 "C22" H 7600 6850 50  0000 L CNN
+F 1 "330nF" H 7600 6550 50  0000 L CNN
+F 2 "Capacitor_SMD:C_1206_3216Metric_Pad1.33x1.80mm_HandSolder" H 7950 6700 50  0001 C CNN
+F 3 "~" H 7950 6700 50  0001 C CNN
+	1    7950 6700
+	1    0    0    -1
+$EndComp
+$Comp
+L Device:D_Zener D2
+U 1 1 60DF1524
+P 8650 6750
+F 0 "D2" V 8604 6830 50  0000 L CNN
+F 1 "3V9" V 8695 6830 50  0000 L CNN
+F 2 "Diode_SMD:D_SOD-123" H 8650 6750 50  0001 C CNN
+F 3 "~" H 8650 6750 50  0001 C CNN
+	1    8650 6750
+	0    1    1    0
+$EndComp
+Wire Wire Line
+	8650 5800 8650 6450
+Wire Wire Line
+	7950 6450 8450 6450
+Connection ~ 8650 6450
+Wire Wire Line
+	8650 6450 8650 6600
+Wire Wire Line
+	8450 6950 7950 6950
+Connection ~ 8450 6950
+Wire Wire Line
+	8450 6600 8450 6450
+Connection ~ 8450 6450
+Wire Wire Line
+	8450 6450 8650 6450
+$Comp
+L pspice:CAP C21
+U 1 1 617DF7FC
+P 7950 2750
+F 0 "C21" H 7650 2900 50  0000 L CNN
+F 1 "330nF" H 7650 2600 50  0000 L CNN
+F 2 "Capacitor_SMD:C_1206_3216Metric_Pad1.33x1.80mm_HandSolder" H 7950 2750 50  0001 C CNN
+F 3 "~" H 7950 2750 50  0001 C CNN
+	1    7950 2750
+	1    0    0    -1
+$EndComp
+Wire Wire Line
+	7950 2500 8450 2500
+Wire Wire Line
+	7950 3000 8450 3000
+Connection ~ 8650 3000
+Wire Wire Line
+	8650 3000 8650 3650
+Wire Wire Line
+	8650 2850 8650 3000
+Wire Wire Line
+	8450 2850 8450 3000
+Connection ~ 8450 3000
+Wire Wire Line
+	8450 3000 8650 3000
+$Comp
+L pspice:CAP C20
+U 1 1 618164E6
+P 7150 6650
+F 0 "C20" H 7250 6800 50  0000 L CNN
+F 1 "22pF" H 7250 6500 50  0000 L CNN
+F 2 "Resistor_SMD:R_0805_2012Metric_Pad1.20x1.40mm_HandSolder" H 7150 6650 50  0001 C CNN
+F 3 "~" H 7150 6650 50  0001 C CNN
+	1    7150 6650
+	1    0    0    -1
+$EndComp
+Wire Wire Line
+	7150 6900 7150 7250
+Wire Wire Line
+	7150 7250 6800 7250
+Connection ~ 6800 7250
+Wire Wire Line
+	7150 6400 6800 6400
+Connection ~ 6800 6400
+Wire Wire Line
+	6800 6400 6800 6450
+$Comp
+L pspice:CAP C19
+U 1 1 6184DA29
+P 7150 2650
+F 0 "C19" H 7250 2800 50  0000 L CNN
+F 1 "22pF" H 7250 2500 50  0000 L CNN
+F 2 "Resistor_SMD:R_0805_2012Metric_Pad1.20x1.40mm_HandSolder" H 7150 2650 50  0001 C CNN
+F 3 "~" H 7150 2650 50  0001 C CNN
+	1    7150 2650
+	1    0    0    -1
+$EndComp
+Wire Wire Line
+	7150 2950 6800 2950
+Wire Wire Line
+	6650 2100 6800 2100
+Wire Wire Line
+	6800 2800 6800 2950
+Connection ~ 6800 2950
+Wire Wire Line
+	6800 2950 6800 3750
+Wire Wire Line
+	6800 2500 6800 2100
+Connection ~ 6800 2100
+Wire Wire Line
+	6800 2100 7150 2100
+Wire Wire Line
+	7150 2100 7150 2400
+Wire Wire Line
+	7150 2900 7150 2950
 $EndSCHEMATC
