File: cntrl_board/codec.sch (KiCad schematic (older format))
At the start: 159 parts, among them J14 Left, J15 Right, J16 Conn_01x03_Male, J17 Conn_01x03_Male, J18 ch5, J19 ch6, J20 ch1, J21 ch2, J22 ch3, J23 ch4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

Commit message: update xformer soft startup
Parts:
- R56: value 10K -> 1K
- U7: symbol ad1937:AD1937WBSTZ -> controller-rescue:AD1937WBSTZ-ad1937
Changed lines of the file:
@@
 	1550 2400 1950 2400
 $Comp
-L ad1937:AD1937WBSTZ U?
+L controller-rescue:AD1937WBSTZ-ad1937 U?
 U 1 1 60CBDFB2
 P 1950 1400
 AR Path="/60BF255D/60CBDFB2" Ref="U?"  Part="1"
 AR Path="/60CBC38F/60CBDFB2" Ref="U7"  Part="1"
+AR Path="/60CBDFB2" Ref="U7"  Part="1"
 F 0 "U7" H 3250 1887 60  0000 C CNN
 F 1 "AD1937WBSTZ" H 3250 1781 60  0000 C CNN
@@
 $EndComp
 $Comp
-L ad1937:AD1937WBSTZ U7
+L controller-rescue:AD1937WBSTZ-ad1937 U7
 U 2 1 60EC66AE
 P 9450 8450
+AR Path="/60EC66AE" Ref="U7"  Part="2"
+AR Path="/60CBC38F/60EC66AE" Ref="U7"  Part="2"
 F 0 "U7" H 9850 6200 60  0000 L CNN
 F 1 "AD1937WBSTZ" H 9850 6100 60  0000 L CNN
@@
 P 7250 1800
 F 0 "R56" V 7300 1950 50  0000 L CNN
-F 1 "10K" V 7250 1700 50  0000 L CNN
+F 1 "1K" V 7250 1700 50  0000 L CNN
 F 2 "Resistor_SMD:R_0603_1608Metric_Pad0.98x0.95mm_HandSolder" V 7180 1800 50  0001 C CNN
 F 3 "~" H 7250 1800 50  0001 C CNN
